Commit message: contact sensors have been added to all the fingers

File: inmoov_description/urdf/leftHand.urdf.xacro (robot description, xacro)
@@ -79,5 +79,5 @@
       </material>
     </visual>
-    <collision>
+    <collision name='lthumb_collision'>
       <geometry>
         <mesh filename="package://inmoov_description/meshes/thumb5_3.stl" scale="0.001 0.001 0.001"/>
@@ -145,5 +145,5 @@
       </material>
     </visual>
-    <collision>
+    <collision name='lindex_collision'>
       <geometry>
         <mesh filename="package://inmoov_description/meshes/index3_3.stl" scale="0.001 0.001 0.001"/>
@@ -211,5 +211,5 @@
       </material>
     </visual>
-    <collision>
+    <collision name='lmiddle_collision'>
       <geometry>
         <mesh filename="package://inmoov_description/meshes/middle3_3.stl" scale="0.001 0.001 0.001"/>
@@ -299,5 +299,5 @@
       </material>
     </visual>
-    <collision>
+    <collision name='lring_collision'>
       <geometry>
         <mesh filename="package://inmoov_description/meshes/ring3_4.stl" scale="0.001 0.001 0.001"/>
@@ -387,5 +387,5 @@
       </material>
     </visual>
-    <collision>
+    <collision name='lpinky_collision'>
       <geometry>
         <mesh filename="package://inmoov_description/meshes/pinky3_4.stl" scale="0.001 0.001 0.001"/>

File: inmoov_description/urdf/rightHand.urdf.xacro (robot description, xacro)
@@ -79,5 +79,5 @@
       </material>
     </visual>
-    <collision>
+    <collision name='rthumb_collision'>
       <geometry>
         <mesh filename="package://inmoov_description/meshes/thumb5_3.stl" scale="0.001 0.001 0.001"/>
@@ -145,5 +145,5 @@
       </material>
     </visual>
-    <collision>
+    <collision name='rindex_collision'>
       <geometry>
         <mesh filename="package://inmoov_description/meshes/index3_3.stl" scale="0.001 0.001 0.001"/>
@@ -211,5 +211,5 @@
       </material>
     </visual>
-    <collision>
+    <collision name='rmiddle_collision'>
       <geometry>
         <mesh filename="package://inmoov_description/meshes/middle3_3.stl" scale="0.001 0.001 0.001"/>
@@ -299,5 +299,5 @@
       </material>
     </visual>
-    <collision>
+    <collision name='rring_collision'>
       <geometry>
         <mesh filename="package://inmoov_description/meshes/ring3_4.stl" scale="0.001 0.001 0.001"/>
@@ -387,5 +387,5 @@
       </material>
     </visual>
-    <collision>
+    <collision name='rpinky_collision'>
       <geometry>
         <mesh filename="package://inmoov_description/meshes/pinky3_4.stl" scale="0.001 0.001 0.001"/>
