Commit message: this isn't working (model explodes), but going to save work and then go back to prev. tag to make sure things before this commit still work...

File: inmoov_description/robots/inmoov.urdf (robot description, URDF)
Before this commit: robot inmoov, 88 links, 87 joints
Links:
- link chestplate: mass 1 -> 0.07
- link disk: mass 1 -> 0.0976
- link eyesupport: mass 1 -> 0.0147
- link face: mass 1 -> 0.01437
- link head: mass 1 -> 0.1
- link head_base: mass 1 -> 0.023
- link jaw: mass 1 -> 0.031
- link kinect: mass 1 -> 1.3
- link left_bicep: mass 1 -> 0.148
- link left_bicepcover: mass 1 -> 0.15
- link left_camera: mass 1 -> 0.026
- link left_cover_handpinky: mass 1 -> 0.002
- link left_cover_handring: mass 1 -> 0.002
- link left_cover_index: mass 1 -> 0.002
- link left_cover_middle: mass 1 -> 0.002
- link left_cover_pinky: mass 1 -> 0.002
- link left_cover_ring: mass 1 -> 0.002
- link left_cover_thumb: mass 1 -> 0.002
- link left_ear: mass 1 -> 0.045
- link left_eye: mass 1 -> 0.0026
- link left_eyesupport: mass 1 -> 0.01
- link left_forearm: mass 1 -> 0.06
- link left_hand: mass 1 -> 0.044
- link left_handcover: mass 1 -> 0.023
- link left_index1: mass 1 -> 0.003
- link left_index2: mass 1 -> 0.003
- link left_index3: mass 1 -> 0.003
- link left_iris: mass 1 -> 0.0005
- link left_middle1: mass 1 -> 0.003
- link left_middle2: mass 1 -> 0.003
- link left_middle3: mass 1 -> 0.003
- link left_pinky1: mass 1 -> 0.003
- link left_pinky2: mass 1 -> 0.003
- link left_pinky3: mass 1 -> 0.003
- link left_pinky4: mass 1 -> 0.003
- link left_ring1: mass 1 -> 0.003
- link left_ring2: mass 1 -> 0.003
- link left_ring3: mass 1 -> 0.003
- link left_ring4: mass 1 -> 0.003
- link left_shoulder: mass 1 -> 0.15
- link left_shoulder_base: mass 1 -> 0.25
- link left_thumb1: mass 1 -> 0.005
- link left_thumb2: mass 1 -> 0.004
- link left_thumb3: mass 1 -> 0.003
- link mid_stomach: mass 1 -> 0.75
- link pedestal: mass 10 -> 1
- link right_bicep: mass 1 -> 0.148
- link right_bicepcover: mass 1 -> 0.15
- link right_camera: mass 1 -> 0.026
- link right_cover_handpinky: mass 1 -> 0.002
- link right_cover_handring: mass 1 -> 0.002
- link right_cover_index: mass 1 -> 0.002
- link right_cover_middle: mass 1 -> 0.002
- link right_cover_pinky: mass 1 -> 0.002
- link right_cover_ring: mass 1 -> 0.002
- link right_cover_thumb: mass 1 -> 0.002
- link right_ear: mass 1 -> 0.045
- link right_eye: mass 1 -> 0.0026
- link right_eyesupport: mass 1 -> 0.01
- link right_forearm: mass 1 -> 0.06
- link right_hand: mass 1 -> 0.044
- link right_handcover: mass 1 -> 0.023
- link right_index1: mass 1 -> 0.003
- link right_index2: mass 1 -> 0.003
- link right_index3: mass 1 -> 0.003
- link right_iris: mass 1 -> 0.0005
- link right_middle1: mass 1 -> 0.003
- link right_middle2: mass 1 -> 0.003
- link right_middle3: mass 1 -> 0.003
- link right_pinky1: mass 1 -> 0.003
- link right_pinky2: mass 1 -> 0.003
- link right_pinky3: mass 1 -> 0.003
- link right_pinky4: mass 1 -> 0.003
- link right_ring1: mass 1 -> 0.003
- link right_ring2: mass 1 -> 0.003
- link right_ring3: mass 1 -> 0.003
- link right_ring4: mass 1 -> 0.003
- link right_shoulder: mass 1 -> 0.15
- link right_shoulder_base: mass 1 -> 0.25
- link right_thumb1: mass 1 -> 0.005
- link right_thumb2: mass 1 -> 0.004
- link right_thumb3: mass 1 -> 0.003
- link skull: mass 1 -> 0.066
- link top_stomach: mass 1 -> 0.75
- link torso: mass 1 -> 5.95

File: inmoov_description/robots/inmoov.urdf.xacro (robot description, xacro)
@@ -49,6 +49,6 @@
     <inertial>
       <origin rpy="0 0 0" xyz="0 0 0.58"/>
-      <mass value="10"/>
-      <inertia ixx="1"  ixy="0"  ixz="0" iyy="1" iyz="0" izz="1" />
+      <mass value="1"/>
+      <inertia ixx="0.01"  ixy="0"  ixz="0" iyy="0.01" iyz="0" izz="0.01" />
     </inertial>
   </link>
@@ -70,5 +70,5 @@
       <origin rpy="0 0 0" xyz="0 0 0"/>
       <mass value="1"/>
-      <inertia ixx="0.1"  ixy="0"  ixz="0" iyy="0.1" iyz="0" izz="0.1" />
+      <inertia ixx="0.0001"  ixy="0"  ixz="0" iyy="0.0001" iyz="0" izz="0.0001" />
     </inertial>
   </link>

File: inmoov_description/urdf/asmArm.urdf.xacro (robot description, xacro)
@@ -19,6 +19,6 @@
     <inertial>
       <origin rpy="0 0 0" xyz="0 0 0"/>
-      <mass value="1"/>
-      <inertia ixx="0.1"  ixy="0"  ixz="0" iyy="0.1" iyz="0" izz="0.1" />
+      <mass value="0.25"/>
+      <inertia ixx="0.0019"  ixy="0"  ixz="0" iyy="0.0018" iyz="0" izz="0.0012" />
     </inertial>
   </link>
@@ -39,6 +39,6 @@
     <inertial>
       <origin rpy="0 0 0" xyz="0 0 0"/>
-      <mass value="1"/>
-      <inertia ixx="0.1"  ixy="0"  ixz="0" iyy="0.1" iyz="0" izz="0.1" />
+      <mass value="0.15"/>
+      <inertia ixx="0.0014"  ixy="0"  ixz="0" iyy="0.0001" iyz="0" izz="0.0014" />
     </inertial>
   </link>
@@ -59,6 +59,6 @@
     <inertial>
       <origin rpy="0 0 0" xyz="0 0 0"/>
-      <mass value="1"/>
-      <inertia ixx="0.1"  ixy="0"  ixz="0" iyy="0.1" iyz="0" izz="0.1" />
+      <mass value="0.148"/>
+      <inertia ixx="0.0007"  ixy="0"  ixz="0" iyy="0.0007" iyz="0" izz="0.0002" />
     </inertial>
   </link>
@@ -79,6 +79,6 @@
     <inertial>
       <origin rpy="0 0 0" xyz="0 0 0"/>
-      <mass value="1"/>
-      <inertia ixx="0.1"  ixy="0"  ixz="0" iyy="0.1" iyz="0" izz="0.1" />
+      <mass value="0.15"/>
+      <inertia ixx="0.0040"  ixy="0"  ixz="0" iyy="0.0035" iyz="0" izz="0.0025" />
     </inertial>
   </link>
@@ -99,6 +99,6 @@
     <inertial>
       <origin rpy="0 0 0" xyz="${flip * 0.001} 0 0"/>
-      <mass value="1"/>
-      <inertia ixx="0.1"  ixy="0"  ixz="0" iyy="0.1" iyz="0" izz="0.1" />
+      <mass value="0.06"/>
+      <inertia ixx="0.0033"  ixy="0"  ixz="0" iyy="0.0033" iyz="0" izz="0.0007" />
     </inertial>
   </link>

File: inmoov_description/urdf/asmFace.urdf.xacro (robot description, xacro)
@@ -19,6 +19,6 @@
     <inertial>
       <origin rpy="0 0 0" xyz="0 0 0" />
-      <mass value="1"/>
-      <inertia ixx="0.1"  ixy="0"  ixz="0" iyy="0.1" iyz="0" izz="0.1" />
+      <mass value="0.01437"/>
+      <inertia ixx="0.0003"  ixy="0"  ixz="0" iyy="0.0015" iyz="0" izz="0.0013" />
     </inertial>
   </link>
@@ -47,6 +47,6 @@
     <inertial>
       <origin rpy="0 0 0" xyz="0 0 0" />
-      <mass value="1"/>
-      <inertia ixx="0.1"  ixy="0"  ixz="0" iyy="0.1" iyz="0" izz="0.1" />
+      <mass value="0.0147"/>
+      <inertia ixx="0.0001"  ixy="0"  ixz="0" iyy="0.0001" iyz="0" izz="0.0001" />
     </inertial>
   </link>
@@ -88,6 +88,6 @@
     <inertial>
       <origin rpy="0 0 0" xyz="0 0 0" />
-      <mass value="1"/>
-      <inertia ixx="0.1"  ixy="0"  ixz="0" iyy="0.1" iyz="0" izz="0.1" />
+      <mass value="0.01"/>
+      <inertia ixx="0.0001"  ixy="0"  ixz="0" iyy="0.0001" iyz="0" izz="0.0001" />
     </inertial>
   </link>
@@ -108,6 +108,6 @@
     <inertial>
       <origin rpy="0 0 0" xyz="0 0 0" />
-      <mass value="1"/>
-      <inertia ixx="0.1"  ixy="0"  ixz="0" iyy="0.1" iyz="0" izz="0.1" />
+      <mass value="0.026"/>
+      <inertia ixx="0.0001"  ixy="0"  ixz="0" iyy="0.0001" iyz="0" izz="0.0001" />
     </inertial>
   </link>
@@ -128,6 +128,6 @@
     <inertial>
       <origin rpy="0 0 0" xyz="0 0 0" />
-      <mass value="1"/>
-      <inertia ixx="0.1"  ixy="0"  ixz="0" iyy="0.1" iyz="0" izz="0.1" />
+      <mass value="0.0026"/>
+      <inertia ixx="0.0001"  ixy="0"  ixz="0" iyy="0.0001" iyz="0" izz="0.0001" />
     </inertial>
   </link>
@@ -148,6 +148,6 @@
     <inertial>
       <origin rpy="0 0 0" xyz="0 0 0" />
-      <mass value="1"/>
-      <inertia ixx="0.1"  ixy="0"  ixz="0" iyy="0.1" iyz="0" izz="0.1" />
+      <mass value="0.0005"/>
+      <inertia ixx="0.0001"  ixy="0"  ixz="0" iyy="0.0001" iyz="0" izz="0.0001" />
     </inertial>
   </link>

File: inmoov_description/urdf/asmHand.urdf.xacro (robot description, xacro)
@@ -19,6 +19,6 @@
     <inertial>
       <origin rpy="0 0 0" xyz="0 0 0"/>
-      <mass value="1"/>
-      <inertia ixx="0.1"  ixy="0"  ixz="0" iyy="0.1" iyz="0" izz="0.1" />
+      <mass value="0.044"/>
+      <inertia ixx="0.0001"  ixy="0"  ixz="0" iyy="0.0007" iyz="0" izz="0.0001" />
     </inertial>
   </link>
@@ -39,6 +39,6 @@
     <inertial>
       <origin rpy="3.1415 0 0" xyz="0 0 0"/>
-      <mass value="1"/>
-      <inertia ixx="0.1"  ixy="0"  ixz="0" iyy="0.1" iyz="0" izz="0.1" />
+      <mass value="0.005"/>
+      <inertia ixx="0.0001"  ixy="0"  ixz="0" iyy="0.0001" iyz="0" izz="0.0001" />
     </inertial>
   </link>
@@ -59,6 +59,6 @@
     <inertial>
       <origin rpy="0 0 3.1415" xyz="0 0 0"/>
-      <mass value="1"/>
-      <inertia ixx="0.1"  ixy="0"  ixz="0" iyy="0.1" iyz="0" izz="0.1" />
+      <mass value="0.004"/>
+      <inertia ixx="0.0001"  ixy="0"  ixz="0" iyy="0.0001" iyz="0" izz="0.0001" />
     </inertial>
   </link>
@@ -79,6 +79,6 @@
     <inertial>
       <origin rpy="0 0 3.1415" xyz="0 0 0"/>
-      <mass value="1"/>
-      <inertia ixx="0.1"  ixy="0"  ixz="0" iyy="0.1" iyz="0" izz="0.1" />
+      <mass value="0.003"/>
+      <inertia ixx="0.0001"  ixy="0"  ixz="0" iyy="0.0001" iyz="0" izz="0.0001" />
     </inertial>
   </link>
@@ -99,6 +99,6 @@
     <inertial>
       <origin rpy="0 0 3.1415" xyz="0 0 0"/>
-      <mass value="1"/>
-      <inertia ixx="0.1"  ixy="0"  ixz="0" iyy="0.1" iyz="0" izz="0.1" />
+      <mass value="0.003"/>
+      <inertia ixx="0.0001"  ixy="0"  ixz="0" iyy="0.0001" iyz="0" izz="0.0001" />
     </inertial>
   </link>
@@ -119,6 +119,6 @@
     <inertial>
       <origin rpy="0 0 3.1415" xyz="0 0 0"/>
-      <mass value="1"/>
-      <inertia ixx="0.1"  ixy="0"  ixz="0" iyy="0.1" iyz="0" izz="0.1" />
+      <mass value="0.003"/>
+      <inertia ixx="0.0001"  ixy="0"  ixz="0" iyy="0.0001" iyz="0" izz="0.0001" />
     </inertial>
   </link>
@@ -139,6 +139,6 @@
     <inertial>
       <origin rpy="0 0 3.1415" xyz="0 0 0"/>
-      <mass value="1"/>
-      <inertia ixx="0.1"  ixy="0"  ixz="0" iyy="0.1" iyz="0" izz="0.1" />
+      <mass value="0.003"/>
+      <inertia ixx="0.0001"  ixy="0"  ixz="0" iyy="0.0001" iyz="0" izz="0.0001" />
     </inertial>
   </link>
@@ -159,6 +159,6 @@
     <inertial>
       <origin rpy="0 0 3.1415" xyz="0 0 0"/>
-      <mass value="1"/>
-      <inertia ixx="0.1"  ixy="0"  ixz="0" iyy="0.1" iyz="0" izz="0.1" />
+      <mass value="0.003"/>
+      <inertia ixx="0.0001"  ixy="0"  ixz="0" iyy="0.0001" iyz="0" izz="0.0001" />
     </inertial>
   </link>
@@ -179,6 +179,6 @@
     <inertial>
       <origin rpy="0 0 3.1415" xyz="0 0 0"/>
-      <mass value="1"/>
-      <inertia ixx="0.1"  ixy="0"  ixz="0" iyy="0.1" iyz="0" izz="0.1" />
+      <mass value="0.003"/>
+      <inertia ixx="0.0001"  ixy="0"  ixz="0" iyy="0.0001" iyz="0" izz="0.0001" />
     </inertial>
   </link>
@@ -199,6 +199,6 @@
     <inertial>
       <origin rpy="0 0 3.1415" xyz="0 0 0"/>
-      <mass value="1"/>
-      <inertia ixx="0.1"  ixy="0"  ixz="0" iyy="0.1" iyz="0" izz="0.1" />
+      <mass value="0.003"/>
+      <inertia ixx="0.0001"  ixy="0"  ixz="0" iyy="0.0001" iyz="0" izz="0.0001" />
     </inertial>
   </link>
@@ -219,6 +219,6 @@
     <inertial>
       <origin rpy="0 0 3.1415" xyz="0 0 0"/>
-      <mass value="1"/>
-      <inertia ixx="0.1"  ixy="0"  ixz="0" iyy="0.1" iyz="0" izz="0.1" />
+      <mass value="0.003"/>
+      <inertia ixx="0.0001"  ixy="0"  ixz="0" iyy="0.0001" iyz="0" izz="0.0001" />
     </inertial>
   </link>
@@ -239,6 +239,6 @@
     <inertial>
       <origin rpy="0 0 3.1415" xyz="0 0 0"/>
-      <mass value="1"/>
-      <inertia ixx="0.1"  ixy="0"  ixz="0" iyy="0.1" iyz="0" izz="0.1" />
+      <mass value="0.003"/>
+      <inertia ixx="0.0001"  ixy="0"  ixz="0" iyy="0.0001" iyz="0" izz="0.0001" />
     </inertial>
   </link>
@@ -259,6 +259,6 @@
     <inertial>
       <origin rpy="0 0 3.1415" xyz="0 0 0"/>
-      <mass value="1"/>
-      <inertia ixx="0.1"  ixy="0"  ixz="0" iyy="0.1" iyz="0" izz="0.1" />
+      <mass value="0.003"/>
+      <inertia ixx="0.0001"  ixy="0"  ixz="0" iyy="0.0001" iyz="0" izz="0.0001" />
     </inertial>
   </link>
@@ -279,6 +279,6 @@
     <inertial>
       <origin rpy="0 0 3.1415" xyz="0 0 0"/>
-      <mass value="1"/>
-      <inertia ixx="0.1"  ixy="0"  ixz="0" iyy="0.1" iyz="0" izz="0.1" />
+      <mass value="0.003"/>
+      <inertia ixx="0.0001"  ixy="0"  ixz="0" iyy="0.0001" iyz="0" izz="0.0001" />
     </inertial>
   </link>
@@ -299,6 +299,6 @@
     <inertial>
       <origin rpy="0 0 3.1415" xyz="0 0 0"/>
-      <mass value="1"/>
-      <inertia ixx="0.1"  ixy="0"  ixz="0" iyy="0.1" iyz="0" izz="0.1" />
+      <mass value="0.003"/>
+      <inertia ixx="0.0001"  ixy="0"  ixz="0" iyy="0.0001" iyz="0" izz="0.0001" />
     </inertial>
   </link>
@@ -319,6 +319,6 @@
     <inertial>
       <origin rpy="0 0 3.1415" xyz="0 0 0"/>
-      <mass value="1"/>
-      <inertia ixx="0.1"  ixy="0"  ixz="0" iyy="0.1" iyz="0" izz="0.1" />
+      <mass value="0.003"/>
+      <inertia ixx="0.0001"  ixy="0"  ixz="0" iyy="0.0001" iyz="0" izz="0.0001" />
     </inertial>
   </link>
@@ -339,6 +339,6 @@
     <inertial>
       <origin rpy="0 0 3.1415" xyz="0 0 0"/>
-      <mass value="1"/>
-      <inertia ixx="0.1"  ixy="0"  ixz="0" iyy="0.1" iyz="0" izz="0.1" />
+      <mass value="0.003"/>
+      <inertia ixx="0.0001"  ixy="0"  ixz="0" iyy="0.0001" iyz="0" izz="0.0001" />
     </inertial>
   </link>
@@ -359,6 +359,6 @@
     <inertial>
       <origin rpy="0 0 3.1415" xyz="0 0 0"/>
-      <mass value="1"/>
-      <inertia ixx="0.1"  ixy="0"  ixz="0" iyy="0.1" iyz="0" izz="0.1" />
+      <mass value="0.003"/>
+      <inertia ixx="0.0001"  ixy="0"  ixz="0" iyy="0.0001" iyz="0" izz="0.0001" />
     </inertial>
   </link>
@@ -370,4 +370,5 @@
    <parent link="${side}_hand"/>
    <child link="${side}_thumb1"/>
+   <dynamics damping="0.7"/>
   </joint>
   <joint name="${side}_thumb" type="revolute">
@@ -386,4 +387,5 @@
    <parent link="${side}_thumb2"/>
    <child link="${side}_thumb3"/>
+   <dynamics damping="0.7"/>
   </joint>
   <joint name="${side}_index1" type="revolute">
@@ -394,4 +396,5 @@
    <parent link="${side}_hand"/>
    <child link="${side}_index1"/>
+   <dynamics damping="0.7"/>
   </joint>
   <joint name="${side}_index" type="revolute">
@@ -410,4 +413,5 @@
    <parent link="${side}_index2"/>
    <child link="${side}_index3"/>
+   <dynamics damping="0.7"/>
   </joint>
   <joint name="${side}_middle1" type="revolute">
@@ -418,4 +422,5 @@
    <parent link="${side}_hand"/>
    <child link="${side}_middle1"/>
+   <dynamics damping="0.7"/>
   </joint>
   <joint name="${side}_middle" type="revolute">
@@ -434,4 +439,5 @@
    <parent link="${side}_middle2"/>
    <child link="${side}_middle3"/>
+   <dynamics damping="0.7"/>
   </joint>
   <joint name="${side}_ring1" type="revolute">
@@ -442,4 +448,5 @@
    <parent link="${side}_hand"/>
    <child link="${side}_ring1"/>
+   <dynamics damping="0.7"/>
   </joint>
   <joint name="${side}_ring" type="revolute">
@@ -458,4 +465,5 @@
    <parent link="${side}_ring2"/>
    <child link="${side}_ring3"/>
+   <dynamics damping="0.7"/>
   </joint>
   <joint name="${side}_ring4" type="revolute">
@@ -466,4 +474,5 @@
    <parent link="${side}_ring3"/>
    <child link="${side}_ring4"/>
+   <dynamics damping="0.7"/>
   </joint>
   <joint name="${side}_pinky1" type="revolute">
@@ -474,4 +483,5 @@
    <parent link="${side}_hand"/>
    <child link="${side}_pinky1"/>
+   <dynamics damping="0.7"/>
   </joint>
   <joint name="${side}_pinky" type="revolute">
@@ -490,4 +500,5 @@
    <parent link="${side}_pinky2"/>
    <child link="${side}_pinky3"/>
+   <dynamics damping="0.7"/>
   </joint>
   <joint name="${side}_pinky4" type="revolute">
@@ -498,4 +509,5 @@
    <parent link="${side}_pinky3"/>
    <child link="${side}_pinky4"/>
+   <dynamics damping="0.7"/>
   </joint>
   <link name="${side}_handcover">
@@ -515,6 +527,6 @@
     <inertial>
       <origin rpy="0 0 0" xyz="0 0 0"/>
-      <mass value="1"/>
-      <inertia ixx="0.1"  ixy="0"  ixz="0" iyy="0.1" iyz="0" izz="0.1" />
+      <mass value="0.023"/>
+      <inertia ixx="0.0001"  ixy="0"  ixz="0" iyy="0.0003" iyz="0" izz="0.0001" />
     </inertial>
   </link>
@@ -535,6 +547,6 @@
     <inertial>
       <origin rpy="0 0 3.1415" xyz="0 0 0"/>
-      <mass value="1"/>
-      <inertia ixx="0.1"  ixy="0"  ixz="0" iyy="0.1" iyz="0" izz="0.1" />
+      <mass value="0.002"/>
+      <inertia ixx="0.0001"  ixy="0"  ixz="0" iyy="0.0001" iyz="0" izz="0.0001" />
     </inertial>
   </link>
@@ -555,6 +567,6 @@
     <inertial>
       <origin rpy="0 0 3.1415" xyz="0 0 0"/>
-      <mass value="1"/>
-      <inertia ixx="0.1"  ixy="0"  ixz="0" iyy="0.1" iyz="0" izz="0.1" />
+      <mass value="0.002"/>
+      <inertia ixx="0.0001"  ixy="0"  ixz="0" iyy="0.0001" iyz="0" izz="0.0001" />
     </inertial>
   </link>
@@ -575,6 +587,6 @@
     <inertial>
       <origin rpy="0 0 3.1415" xyz="0 0 0"/>
-      <mass value="1"/>
-      <inertia ixx="0.1"  ixy="0"  ixz="0" iyy="0.1" iyz="0" izz="0.1" />
+      <mass value="0.002"/>
+      <inertia ixx="0.0001"  ixy="0"  ixz="0" iyy="0.0001" iyz="0" izz="0.0001" />
     </inertial>
   </link>
@@ -595,6 +607,6 @@
     <inertial>
       <origin rpy="0 0 3.1415" xyz="0 0 0"/>
-      <mass value="1"/>
-      <inertia ixx="0.1"  ixy="0"  ixz="0" iyy="0.1" iyz="0" izz="0.1" />
+      <mass value="0.002"/>
+      <inertia ixx="0.0001"  ixy="0"  ixz="0" iyy="0.0001" iyz="0" izz="0.0001" />
     </inertial>
   </link>
@@ -615,6 +627,6 @@
     <inertial>
       <origin rpy="0 0 3.1415" xyz="0 0 0"/>
-      <mass value="1"/>
-      <inertia ixx="0.1"  ixy="0"  ixz="0" iyy="0.1" iyz="0" izz="0.1" />
+      <mass value="0.002"/>
+      <inertia ixx="0.0001"  ixy="0"  ixz="0" iyy="0.0001" iyz="0" izz="0.0001" />
     </inertial>
   </link>
@@ -635,6 +647,6 @@
     <inertial>
       <origin rpy="0 0 3.1415" xyz="0 0 0"/>
-      <mass value="1"/>
-      <inertia ixx="0.1"  ixy="0"  ixz="0" iyy="0.1" iyz="0" izz="0.1" />
+      <mass value="0.002"/>
+      <inertia ixx="0.0001"  ixy="0"  ixz="0" iyy="0.0001" iyz="0" izz="0.0001" />
     </inertial>
   </link>
@@ -655,6 +667,6 @@
     <inertial>
       <origin rpy="0 0 3.1415" xyz="0 0 0"/>
-      <mass value="1"/>
-      <inertia ixx="0.1"  ixy="0"  ixz="0" iyy="0.1" iyz="0" izz="0.1" />
+      <mass value="0.002"/>
+      <inertia ixx="0.0001"  ixy="0"  ixz="0" iyy="0.0001" iyz="0" izz="0.0001" />
     </inertial>
   </link>

File: inmoov_description/urdf/asmHead.urdf.xacro (robot description, xacro)
@@ -19,6 +19,6 @@
     <inertial>
       <origin rpy="0 0 0" xyz="0 0 0" />
-      <mass value="1"/>
-      <inertia ixx="0.1"  ixy="0"  ixz="0" iyy="0.1" iyz="0" izz="0.1" />
+      <mass value="0.023"/>
+      <inertia ixx="0.0001"  ixy="0"  ixz="0" iyy="0.0001" iyz="0" izz="0.0001" />
     </inertial>
   </link>
@@ -39,6 +39,6 @@
     <inertial>
       <origin rpy="0 0 0" xyz="0 0 0" />
-      <mass value="1"/>
-      <inertia ixx="0.1"  ixy="0"  ixz="0" iyy="0.1" iyz="0" izz="0.1" />
+      <mass value="0.1"/>
+      <inertia ixx="0.0001"  ixy="0"  ixz="0" iyy="0.0001" iyz="0" izz="0.0001" />
     </inertial>
   </link>
@@ -59,6 +59,6 @@
     <inertial>
       <origin rpy="0 0 3.1415" xyz="0 0 0" />
-      <mass value="1"/>
-      <inertia ixx="0.1"  ixy="0"  ixz="0" iyy="0.1" iyz="0" izz="0.1" />
+      <mass value="0.031"/>
+      <inertia ixx="0.0001"  ixy="0"  ixz="0" iyy="0.0001" iyz="0" izz="0.0001" />
     </inertial>
   </link>
@@ -79,6 +79,6 @@
     <inertial>
       <origin rpy="0 0 0" xyz="0.001 0 0" />
-      <mass value="1"/>
-      <inertia ixx="0.1"  ixy="0"  ixz="0" iyy="0.1" iyz="0" izz="0.1" />
+      <mass value="0.066"/>
+      <inertia ixx="0.0034"  ixy="0"  ixz="0" iyy="0.0024" iyz="0" izz="0.0029" />
     </inertial>
   </link>
@@ -99,6 +99,6 @@
     <inertial>
       <origin rpy="0 0 0" xyz="0 0 0" />
-      <mass value="1"/>
-      <inertia ixx="0.1"  ixy="0"  ixz="0" iyy="0.1" iyz="0" izz="0.1" />
+      <mass value="0.045"/>
+      <inertia ixx="0.0001"  ixy="0"  ixz="0" iyy="0.0001" iyz="0" izz="0.0001" />
     </inertial>
   </link>
@@ -119,6 +119,6 @@
     <inertial>
       <origin rpy="0 0 0" xyz="0 0 0" />
-      <mass value="1"/>
-      <inertia ixx="0.1"  ixy="0"  ixz="0" iyy="0.1" iyz="0" izz="0.1" />
+      <mass value="0.045"/>
+      <inertia ixx="0.0001"  ixy="0"  ixz="0" iyy="0.0001" iyz="0" izz="0.0001" />
     </inertial>
   </link>

File: inmoov_description/urdf/asmTorso.urdf.xacro (robot description, xacro)
@@ -19,6 +19,6 @@
     <inertial>
       <origin rpy="0 0 0" xyz="0 0 1.152"/>
-      <mass value="1"/>
-      <inertia ixx="0.1"  ixy="0"  ixz="0" iyy="0.1" iyz="0" izz="0.1" />
+      <mass value="0.75"/>
+      <inertia ixx="0.0130"  ixy="0"  ixz="0" iyy="0.0271" iyz="0" izz="0.0294" />
     </inertial>
   </link>
@@ -39,6 +39,6 @@
     <inertial>
       <origin rpy="0 0 0" xyz="0 0.046 0"/>
-      <mass value="1"/>
-      <inertia ixx="0.1"  ixy="0"  ixz="0" iyy="0.1" iyz="0" izz="0.1" />
+      <mass value="0.0976"/>
+      <inertia ixx="0.0001"  ixy="0"  ixz="0" iyy="0.0002" iyz="0" izz="0.0001" />
     </inertial>
   </link>
@@ -59,6 +59,6 @@
     <inertial>
       <origin rpy="0 0 0" xyz="0 0 0"/>
-      <mass value="1"/>
-      <inertia ixx="0.1"  ixy="0"  ixz="0" iyy="0.1" iyz="0" izz="0.1" />
+      <mass value="0.75"/>
+      <inertia ixx="0.0099"  ixy="0"  ixz="0" iyy="0.0119" iyz="0" izz="0.0122" />
     </inertial>
   </link>
@@ -79,6 +79,6 @@
     <inertial>
       <origin rpy="0 0 0" xyz="0 0 0"/>
-      <mass value="1"/>
-      <inertia ixx="0.1"  ixy="0"  ixz="0" iyy="0.1" iyz="0" izz="0.1" />
+      <mass value="5.95"/>
+      <inertia ixx="0.0682"  ixy="0"  ixz="0" iyy="0.0808" iyz="0" izz="0.0218" />
     </inertial>
   </link>
@@ -99,6 +99,6 @@
     <inertial>
       <origin rpy="0 0 0" xyz="0 0 0"/>
-      <mass value="1"/>
-      <inertia ixx="0.1"  ixy="0"  ixz="0" iyy="0.1" iyz="0" izz="0.1" />
+      <mass value="1.3"/>
+      <inertia ixx="0.0083"  ixy="0"  ixz="0" iyy="0.0634" iyz="0" izz="0.0644" />
     </inertial>
   </link>
@@ -119,6 +119,6 @@
     <inertial>
       <origin rpy="0 0 0" xyz="0 0 0"/>
-      <mass value="1"/>
-      <inertia ixx="0.1"  ixy="0"  ixz="0" iyy="0.1" iyz="0" izz="0.1" />
+      <mass value="0.07"/>
+      <inertia ixx="0.0024"  ixy="0"  ixz="0" iyy="0.0047" iyz="0" izz="0.0024" />
     </inertial>
   </link>
