Commit message: right ring/pinky issueshould be resolved

File: inmoov_description/robots/inmoov.urdf (robot description, URDF)
Before this commit: robot inmoov, 88 links, 87 joints
Joints:
- joint right_ringCMC: limit lower=-1.57 upper=1.57 effort=1.9613 velocity=6.545 -> lower=-1.57 upper=0 effort=1.9613 velocity=6.545
- joint right_ringDIP: limit lower=-1.57 upper=1.57 effort=1.9613 velocity=6.545 -> lower=0 upper=1.57 effort=1.9613 velocity=6.545
- joint right_ringMCP: limit lower=-1.57 upper=1.5 effort=1.9613 velocity=6.545 -> lower=0 upper=1.5 effort=1.9613 velocity=6.545
- joint right_ringPIP: limit lower=-1.57 upper=1.57 effort=1.9613 velocity=6.545 -> lower=0 upper=1.57 effort=1.9613 velocity=6.545

File: inmoov_description/urdf/rightHand.urdf.xacro (robot description, xacro)
@@ -475,5 +475,5 @@
     <limit effort="1.9613" lower="-1.57" upper="0" velocity="6.545"/>
     <origin rpy="0 -0.7 3.1415" xyz="0.00705 0 -0.0794"/>
-    <mimic joint="right_ringMCP" multiplier="-0.1" offset="0"/>
+    <mimic joint="right_ringMCP" multiplier="0.1" offset="0"/>
     <parent link="right_hand"/>
     <child link="right_ring_meta"/>
@@ -507,5 +507,5 @@
     <limit effort="1.9613" lower="-1.57" upper="0" velocity="6.545"/>
     <origin rpy="0 -0.7 3.1415" xyz="0.027 0 -0.0555"/>
-    <mimic joint="right_pinkyMCP" multiplier="-0.1" offset="0"/>
+    <mimic joint="right_pinkyMCP" multiplier="0.1" offset="0"/>
     <parent link="right_hand"/>
     <child link="right_pinky_meta"/>

Commit message: eye cameras and xbox kinect functionality in gazebo added

File: inmoov_description/robots/inmoov.urdf (robot description, URDF)
Before this commit: robot inmoov, 88 links, 87 joints
Links:
- added link kinectIR; visual cylinder length=0.005 radius=0.011
- added link kinectIR_frame; visual cylinder length=0.001 radius=0.001
Joints:
- added joint kinect_ircamera: type fixed, parent kinect, child kinectIR, origin xyz=-0.015 0.08 0.042 rpy=0 0 1.5708
- added joint kinect_ircamera_frame: type fixed, parent kinectIR, child kinectIR_frame, origin xyz=0 0 0 rpy=-1.5708 0 -1.5708
- joint head_leftright: limit lower=-1.57 upper=1.57 effort=2.422 velocity=7.48 -> lower=-1.05 upper=1.05 effort=2.422 velocity=7.48
- joint head_updown: limit lower=-0.30 upper=0.30 effort=2.422 velocity=7.48 -> lower=-1.22 upper=1.22 effort=2.422 velocity=7.48
- joint jaw: limit lower=0 upper=0.15 effort=1.9613 velocity=6.545 -> lower=0 upper=0.261 effort=1.9613 velocity=6.545
- joint left_bicep_rotate: limit lower=-1.57 upper=1.57 effort=2.422 velocity=7.48 -> lower=-0.872 upper=1.57 effort=2.422 velocity=7.48
- joint right_bicep_rotate: limit lower=-1.57 upper=1.57 effort=2.422 velocity=7.48 -> lower=-0.872 upper=1.57 effort=2.422 velocity=7.48
- joint right_pinkyCMC: mimic joint=right_pinkyMCP multiplier=-0.1 offset=0 -> joint=right_pinkyMCP multiplier=0.1 offset=0
- joint right_ringCMC: mimic joint=right_ringMCP multiplier=-0.1 offset=0 -> joint=right_ringMCP multiplier=0.1 offset=0

File: inmoov_description/robots/inmoov.urdf.xacro (robot description, xacro)
@@ -84,5 +84,5 @@
   <joint name="head_updown" type="revolute">
    <axis xyz="1 0 0"/>
-   <limit effort="2.422" lower="-0.30" upper="0.30" velocity="7.48"/>
+   <limit effort="2.422" lower="-1.22" upper="1.22" velocity="7.48"/>
    <origin rpy="0 0 0" xyz="0 0 0"/>
    <parent link="head_tilt"/>

File: inmoov_description/urdf/asmArm.urdf.xacro (robot description, xacro)
@@ -101,5 +101,5 @@
   <joint name="${side}_bicep_rotate" type="revolute">
     <axis xyz="0 0 1"/>
-    <limit effort="2.422" lower="-1.57" upper="1.57" velocity="7.48"/>
+    <limit effort="2.422" lower="-0.872" upper="1.57" velocity="7.48"/>
     <origin rpy="0 0 0" xyz="${flip * 0.066} 0 -0.060"/>
     <parent link="${side}_shoulder"/>

File: inmoov_description/urdf/asmHead.urdf.xacro (robot description, xacro)
@@ -113,5 +113,5 @@
   <joint name="head_leftright" type="revolute">
    <axis xyz="0 0 1"/>
-   <limit effort="2.422" lower="-1.57" upper="1.57" velocity="7.48"/>
+   <limit effort="2.422" lower="-1.05" upper="1.05" velocity="7.48"/>
    <origin rpy="0 0 0" xyz="0 0 0.0245"/>
    <parent link="head_base"/>
@@ -121,5 +121,5 @@
   <joint name="jaw" type="revolute">
    <axis xyz="1 0 0"/>
-   <limit effort="1.9613" lower="0" upper="0.15" velocity="6.545"/>
+   <limit effort="1.9613" lower="0" upper="0.261" velocity="6.545"/>
    <origin rpy="0.085 0 3.1415" xyz="-0.001 0.0375 0.0437"/>
    <parent link="head"/>

File: inmoov_description/urdf/asmTorso.urdf.xacro (robot description, xacro)
@@ -103,4 +103,22 @@
     </inertial>
   </link>
+  <link name="kinectIR">
+    <visual>
+      <geometry>
+        <cylinder length="0.005" radius="0.011"/>
+      </geometry>
+      <origin rpy="0 1.5708 0" xyz="0 0 0"/>
+      <xacro:frame_color/>
+    </visual>
+  </link>
+  <link name="kinectIR_frame">
+    <visual>
+      <geometry>
+        <cylinder length="0.001" radius="0.001"/>
+      </geometry>
+      <origin rpy="0 0 0" xyz="0 0 0"/>
+      <xacro:frame_color/>
+    </visual>
+  </link>
   <link name="chestplate">
     <visual>
@@ -154,4 +172,14 @@
     <child link="kinect"/>
   </joint>
+  <joint name="kinect_ircamera" type="fixed">
+    <origin rpy="0 0 1.5708" xyz="-0.015 0.08 0.042"/>
+    <parent link="kinect"/>
+    <child link="kinectIR"/>
+  </joint>
+  <joint name="kinect_ircamera_frame" type="fixed">
+    <origin rpy="-1.5708 0 -1.5708" xyz="0 0 0"/>
+    <parent link="kinectIR"/>
+    <child link="kinectIR_frame"/>
+  </joint>
 </xacro:macro>
 </robot>

Commit message: fixed head_base refering to the old location of the meshes folder

File: inmoov_description/robots/inmoov.urdf (robot description, URDF)
Before this commit: robot inmoov, 90 links, 89 joints
Links:
- link head_base: geometry visual mesh filename=package://inmoov_meshes/meshes/head_base.stl scale=0.001 0.001 0.001

File: inmoov_description/urdf/asmHead.urdf.xacro (robot description, xacro)
@@ -6,5 +6,5 @@
     <visual>
       <geometry>
-        <mesh filename="package://inmoov_description/meshes/head_base.stl" scale="0.001 0.001 0.001"/>
+        <mesh filename="package://inmoov_meshes/meshes/head_base.stl" scale="0.001 0.001 0.001"/>
       </geometry>
       <origin rpy="0 0 0" xyz="0 0 0"/>

Commit message: Add a fake joint to each wrist to allow for better moveit group definitions on the arms.

File: inmoov_description/robots/inmoov.urdf (robot description, URDF)
Before this commit: robot inmoov, 90 links, 89 joints
Links:
- added link left_wrist_link, mass 5.25e-4; visual mesh filename=package://inmoov_meshes/meshes/virtual.stl scale=0.001 0.001 0.001
- added link right_wrist_link, mass 5.25e-4; visual mesh filename=package://inmoov_meshes/meshes/virtual.stl scale=0.001 0.001 0.001
Joints:
- added joint left_wrist_fixed: type fixed, parent left_wrist_link, child left_hand, origin xyz=0 0 0 rpy=0 0 0
- added joint right_wrist_fixed: type fixed, parent right_wrist_link, child right_hand, origin xyz=0 0 0 rpy=0 0 0
- joint left_wrist: child left_hand -> left_wrist_link
- joint right_wrist: child right_hand -> right_wrist_link

File: inmoov_description/robots/inmoov.urdf.xacro (robot description, xacro)
@@ -107,4 +107,20 @@
   </joint>
   <xacro:rhand side="right" neg="1" covers="yes" />
+  <link name="right_wrist_link">
+    <visual>
+      <geometry>
+        <mesh filename="package://inmoov_meshes/meshes/virtual.stl" scale="0.001 0.001 0.001"/>
+      </geometry>
+      <origin rpy="0 0 0" xyz="0 0 0"/>
+      <material name="cframe">
+        <color rgba="0.25 0.25 0.25 1"/>
+      </material>
+    </visual>
+    <inertial>
+      <origin rpy="0 0 0" xyz="0 0.001 0.001"/>
+      <mass value="5.25e-4"/>
+      <inertia ixx="1e-3"  ixy="0"  ixz="0" iyy="1e-3" iyz="0" izz="1e-3" />
+    </inertial>
+  </link>
   <joint name="right_wrist" type="revolute">
    <axis xyz="0 0 1"/>
@@ -112,6 +128,11 @@
    <origin rpy="0 0 0" xyz="-0.01 -0.0144 -0.2885"/>
    <parent link="right_forearm"/>
+   <child link="right_wrist_link"/>
+   <dynamics damping="0.7"/>
+  </joint>
+  <joint name="right_wrist_fixed" type="fixed">
+   <origin rpy="0 0 0" xyz="0 0 0"/>
+   <parent link="right_wrist_link"/>
    <child link="right_hand"/>
-   <dynamics damping="0.7"/>
   </joint>
   <xacro:arm side="left" flip="-1" covers="yes" />
@@ -125,4 +146,20 @@
   </joint>
   <xacro:lhand side="left" neg="-1" covers="yes" />
+  <link name="left_wrist_link">
+    <visual>
+      <geometry>
+        <mesh filename="package://inmoov_meshes/meshes/virtual.stl" scale="0.001 0.001 0.001"/>
+      </geometry>
+      <origin rpy="0 0 0" xyz="0 0 0"/>
+      <material name="cframe">
+        <color rgba="0.25 0.25 0.25 1"/>
+      </material>
+    </visual>
+    <inertial>
+      <origin rpy="0 0 0" xyz="0 0.001 0.001"/>
+      <mass value="5.25e-4"/>
+      <inertia ixx="1e-3"  ixy="0"  ixz="0" iyy="1e-3" iyz="0" izz="1e-3" />
+    </inertial>
+  </link>
   <joint name="left_wrist" type="revolute">
    <axis xyz="0 0 1"/>
@@ -130,6 +167,11 @@
    <origin rpy="0 0 0" xyz="0.01 -0.0144 -0.2885"/>
    <parent link="left_forearm"/>
+   <child link="left_wrist_link"/>
+   <dynamics damping="0.7"/>
+  </joint>
+  <joint name="left_wrist_fixed" type="fixed">
+   <origin rpy="0 0 0" xyz="0 0 0"/>
+   <parent link="left_wrist_link"/>
    <child link="left_hand"/>
-   <dynamics damping="0.7"/>
   </joint>
   <xacro:include filename="$(find inmoov_description)/urdf/sensors.gazebo"/>

Commit message: Reflect changes on the 3D-perception branch back to the master branch.

File: inmoov_description/robots/inmoov.urdf (robot description, URDF)
Before this commit: robot inmoov, 90 links, 89 joints
Links:
- added link left_wrist_link, mass 5.25e-4; visual mesh filename=package://inmoov_meshes/meshes/virtual.stl scale=0.001 0.001 0.001
- added link right_wrist_link, mass 5.25e-4; visual mesh filename=package://inmoov_meshes/meshes/virtual.stl scale=0.001 0.001 0.001
Joints:
- added joint left_wrist_fixed: type fixed, parent left_wrist_link, child left_hand, origin xyz=0 0 0 rpy=0 0 0
- added joint right_wrist_fixed: type fixed, parent right_wrist_link, child right_hand, origin xyz=0 0 0 rpy=0 0 0
- joint left_wrist: child left_hand -> left_wrist_link
- joint right_wrist: child right_hand -> right_wrist_link

File: inmoov_description/robots/inmoov.urdf.xacro (robot description, xacro)
@@ -107,4 +107,20 @@
   </joint>
   <xacro:rhand side="right" neg="1" covers="yes" />
+  <link name="right_wrist_link">
+    <visual>
+      <geometry>
+        <mesh filename="package://inmoov_meshes/meshes/virtual.stl" scale="0.001 0.001 0.001"/>
+      </geometry>
+      <origin rpy="0 0 0" xyz="0 0 0"/>
+      <material name="cframe">
+        <color rgba="0.25 0.25 0.25 1"/>
+      </material>
+    </visual>
+    <inertial>
+      <origin rpy="0 0 0" xyz="0 0.001 0.001"/>
+      <mass value="5.25e-4"/>
+      <inertia ixx="1e-3"  ixy="0"  ixz="0" iyy="1e-3" iyz="0" izz="1e-3" />
+    </inertial>
+  </link>
   <joint name="right_wrist" type="revolute">
    <axis xyz="0 0 1"/>
@@ -112,6 +128,11 @@
    <origin rpy="0 0 0" xyz="-0.01 -0.0144 -0.2885"/>
    <parent link="right_forearm"/>
+   <child link="right_wrist_link"/>
+   <dynamics damping="0.7"/>
+  </joint>
+  <joint name="right_wrist_fixed" type="fixed">
+   <origin rpy="0 0 0" xyz="0 0 0"/>
+   <parent link="right_wrist_link"/>
    <child link="right_hand"/>
-   <dynamics damping="0.7"/>
   </joint>
   <xacro:arm side="left" flip="-1" covers="yes" />
@@ -125,4 +146,20 @@
   </joint>
   <xacro:lhand side="left" neg="-1" covers="yes" />
+  <link name="left_wrist_link">
+    <visual>
+      <geometry>
+        <mesh filename="package://inmoov_meshes/meshes/virtual.stl" scale="0.001 0.001 0.001"/>
+      </geometry>
+      <origin rpy="0 0 0" xyz="0 0 0"/>
+      <material name="cframe">
+        <color rgba="0.25 0.25 0.25 1"/>
+      </material>
+    </visual>
+    <inertial>
+      <origin rpy="0 0 0" xyz="0 0.001 0.001"/>
+      <mass value="5.25e-4"/>
+      <inertia ixx="1e-3"  ixy="0"  ixz="0" iyy="1e-3" iyz="0" izz="1e-3" />
+    </inertial>
+  </link>
   <joint name="left_wrist" type="revolute">
    <axis xyz="0 0 1"/>
@@ -130,6 +167,11 @@
    <origin rpy="0 0 0" xyz="0.01 -0.0144 -0.2885"/>
    <parent link="left_forearm"/>
+   <child link="left_wrist_link"/>
+   <dynamics damping="0.7"/>
+  </joint>
+  <joint name="left_wrist_fixed" type="fixed">
+   <origin rpy="0 0 0" xyz="0 0 0"/>
+   <parent link="left_wrist_link"/>
    <child link="left_hand"/>
-   <dynamics damping="0.7"/>
   </joint>
   <xacro:include filename="$(find inmoov_description)/urdf/emr_sensors.gazebo"/>

File: inmoov_description/robots/inmoov_no_collision.urdf (robot description, URDF)
Before this commit: robot inmoov, 90 links, 89 joints
Links:
- added link left_wrist_link, mass 5.25e-4; visual mesh filename=package://inmoov_meshes/meshes/virtual.stl scale=0.001 0.001 0.001
- added link right_wrist_link, mass 5.25e-4; visual mesh filename=package://inmoov_meshes/meshes/virtual.stl scale=0.001 0.001 0.001
Joints:
- added joint left_wrist_fixed: type fixed, parent left_wrist_link, child left_hand, origin xyz=0 0 0 rpy=0 0 0
- added joint right_wrist_fixed: type fixed, parent right_wrist_link, child right_hand, origin xyz=0 0 0 rpy=0 0 0
- joint left_wrist: child left_hand -> left_wrist_link
- joint right_wrist: child right_hand -> right_wrist_link

File: inmoov_description/robots/inmoov_no_collision.urdf.xacro (robot description, xacro)
@@ -95,4 +95,20 @@
   </joint>
   <xacro:rhand side="right" neg="1" covers="yes"/>
+  <link name="right_wrist_link">
+    <visual>
+      <geometry>
+        <mesh filename="package://inmoov_meshes/meshes/virtual.stl" scale="0.001 0.001 0.001"/>
+      </geometry>
+      <origin rpy="0 0 0" xyz="0 0 0"/>
+      <material name="cframe">
+        <color rgba="0.25 0.25 0.25 1"/>
+      </material>
+    </visual>
+    <inertial>
+      <origin rpy="0 0 0" xyz="0 0.001 0.001"/>
+      <mass value="5.25e-4"/>
+      <inertia ixx="1e-3" ixy="0" ixz="0" iyy="1e-3" iyz="0" izz="1e-3"/>
+    </inertial>
+  </link>
   <joint name="right_wrist" type="revolute">
    <axis xyz="0 0 1"/>
@@ -100,6 +116,11 @@
    <origin rpy="0 0 0" xyz="-0.01 -0.0144 -0.2885"/>
    <parent link="right_forearm"/>
+   <child link="right_wrist_link"/>
+   <dynamics damping="0.7"/>
+  </joint>
+  <joint name="right_wrist_fixed" type="fixed">
+   <origin rpy="0 0 0" xyz="0 0 0"/>
+   <parent link="right_wrist_link"/>
    <child link="right_hand"/>
-   <dynamics damping="0.7"/>
   </joint>
   <xacro:arm side="left" flip="-1" covers="yes"/>
@@ -113,4 +134,20 @@
   </joint>
   <xacro:lhand side="left" neg="-1" covers="yes"/>
+  <link name="left_wrist_link">
+    <visual>
+      <geometry>
+        <mesh filename="package://inmoov_meshes/meshes/virtual.stl" scale="0.001 0.001 0.001"/>
+      </geometry>
+      <origin rpy="0 0 0" xyz="0 0 0"/>
+      <material name="cframe">
+        <color rgba="0.25 0.25 0.25 1"/>
+      </material>
+    </visual>
+    <inertial>
+      <origin rpy="0 0 0" xyz="0 0.001 0.001"/>
+      <mass value="5.25e-4"/>
+      <inertia ixx="1e-3" ixy="0" ixz="0" iyy="1e-3" iyz="0" izz="1e-3"/>
+    </inertial>
+  </link>
   <joint name="left_wrist" type="revolute">
    <axis xyz="0 0 1"/>
@@ -118,6 +155,11 @@
    <origin rpy="0 0 0" xyz="0.01 -0.0144 -0.2885"/>
    <parent link="left_forearm"/>
+   <child link="left_wrist_link"/>
+   <dynamics damping="0.7"/>
+  </joint>
+  <joint name="left_wrist_fixed" type="fixed">
+   <origin rpy="0 0 0" xyz="0 0 0"/>
+   <parent link="left_wrist_link"/>
    <child link="left_hand"/>
-   <dynamics damping="0.7"/>
   </joint>
   <xacro:include filename="$(find inmoov_description)/urdf/emr_sensors.gazebo"/>
