Commit message: Changed how the collision-less model is updated and uploaded the actual models.

File: inmoov_description/robots/inmoov.urdf.xacro (robot description, xacro)
@@ -2,11 +2,11 @@
 <robot name="inmoov" xmlns:xacro="http://ros.org/wiki/xacro">
   <xacro:include filename="$(find inmoov_description)/urdf/materials.urdf.xacro" />
-  <xacro:include filename="$(find inmoov_description)/urdf/asmBase.urdf.xacro" />
-  <xacro:include filename="$(find inmoov_description)/urdf/asmTorso.urdf.xacro" />
-  <xacro:include filename="$(find inmoov_description)/urdf/asmHead.urdf.xacro" />
-  <xacro:include filename="$(find inmoov_description)/urdf/asmFace.urdf.xacro" />
-  <xacro:include filename="$(find inmoov_description)/urdf/asmArm.urdf.xacro" />
-  <xacro:include filename="$(find inmoov_description)/urdf/rightHand.urdf.xacro" />
-  <xacro:include filename="$(find inmoov_description)/urdf/leftHand.urdf.xacro" />
+  <xacro:include filename="$(find inmoov_description)/urdf/default/asmBase.urdf.xacro" />
+  <xacro:include filename="$(find inmoov_description)/urdf/default/asmTorso.urdf.xacro" />
+  <xacro:include filename="$(find inmoov_description)/urdf/default/asmHead.urdf.xacro" />
+  <xacro:include filename="$(find inmoov_description)/urdf/default/asmFace.urdf.xacro" />
+  <xacro:include filename="$(find inmoov_description)/urdf/default/asmArm.urdf.xacro" />
+  <xacro:include filename="$(find inmoov_description)/urdf/default/rightHand.urdf.xacro" />
+  <xacro:include filename="$(find inmoov_description)/urdf/default/leftHand.urdf.xacro" />
   <link name="world"/>
   <joint name="fixed" type="fixed">
@@ -133,5 +133,6 @@
    <dynamics damping="0.7"/>
   </joint>
-  <xacro:include filename="$(find inmoov_description)/urdf/sensors.gazebo"/>
+  <xacro:include filename="$(find inmoov_description)/urdf/emr_sensors.gazebo"/>
+  <xacro:include filename="$(find inmoov_description)/urdf/contact_sensors.gazebo"/>
   <xacro:include filename="$(find inmoov_description)/urdf/servos.urdf.xacro"/>
   <xacro:include filename="$(find inmoov_description)/urdf/materials.gazebo"/>

File: inmoov_description/robots/inmoov_no_collision.urdf.xacro (robot description, xacro)
@@ -1,12 +1,12 @@
-<?xml version="1.0"?>
-<robot name="inmoov" xmlns:xacro="http://ros.org/wiki/xacro">
-  <xacro:include filename="$(find inmoov_description)/urdf/materials.urdf.xacro" />
-  <xacro:include filename="$(find inmoov_description)/urdf/asmBase.urdf.xacro" />
-  <xacro:include filename="$(find inmoov_description)/urdf/asmTorso.urdf.xacro" />
-  <xacro:include filename="$(find inmoov_description)/urdf/asmHead.urdf.xacro" />
-  <xacro:include filename="$(find inmoov_description)/urdf/asmFace.urdf.xacro" />
-  <xacro:include filename="$(find inmoov_description)/urdf/asmArm.urdf.xacro" />
-  <xacro:include filename="$(find inmoov_description)/urdf/rightHand.urdf.xacro" />
-  <xacro:include filename="$(find inmoov_description)/urdf/leftHand.urdf.xacro" />
+<?xml version='1.0' encoding='ASCII'?>
+<robot xmlns:xacro="http://ros.org/wiki/xacro" name="inmoov">
+  <xacro:include filename="$(find inmoov_description)/urdf/materials.urdf.xacro"/>
+  <xacro:include filename="$(find inmoov_description)/urdf/no_collisions/asmBase.urdf.xacro"/>
+  <xacro:include filename="$(find inmoov_description)/urdf/no_collisions/asmTorso.urdf.xacro"/>
+  <xacro:include filename="$(find inmoov_description)/urdf/no_collisions/asmHead.urdf.xacro"/>
+  <xacro:include filename="$(find inmoov_description)/urdf/no_collisions/asmFace.urdf.xacro"/>
+  <xacro:include filename="$(find inmoov_description)/urdf/no_collisions/asmArm.urdf.xacro"/>
+  <xacro:include filename="$(find inmoov_description)/urdf/no_collisions/rightHand.urdf.xacro"/>
+  <xacro:include filename="$(find inmoov_description)/urdf/no_collisions/leftHand.urdf.xacro"/>
   <link name="world"/>
   <joint name="fixed" type="fixed">
@@ -22,15 +22,9 @@
       <xacro:base_color/>
     </visual>
-    <collision>
-      <geometry>
-        <cylinder length="0.11" radius="0.26"/>
-      </geometry>
-      <origin rpy="0 0 0" xyz="0 0 0.055"/>
-    </collision>
-  </link>
+    </link>
   <joint name="base_to_pedestal" type="fixed">
     <parent link="base_link"/>
     <child link="pedestal"/>
-    <origin rpy="0 0 0"  xyz="0 0 0"/>
+    <origin rpy="0 0 0" xyz="0 0 0"/>
   </joint>
   <link name="pedestal">
@@ -42,14 +36,8 @@
       <xacro:base_color/>
     </visual>
-    <collision>
-      <geometry>
-        <cylinder length="0.94" radius="0.0254"/>
-      </geometry>
-      <origin rpy="0 0 0" xyz="0 0 0.58"/>
-    </collision>
     <inertial>
       <origin rpy="0 0 0" xyz="0 0 0.58"/>
       <mass value="5"/>
-      <inertia ixx="0.1"  ixy="0"  ixz="0" iyy="0.1" iyz="0" izz="0.1" />
+      <inertia ixx="0.1" ixy="0" ixz="0" iyy="0.1" iyz="0" izz="0.1"/>
     </inertial>
   </link>
@@ -65,5 +53,5 @@
       <origin rpy="0 0 0" xyz="0 0.001 0.001"/>
       <mass value="5.25e-4"/>
-      <inertia ixx="1e-3"  ixy="0"  ixz="0" iyy="1e-3" iyz="0" izz="1e-3" />
+      <inertia ixx="1e-3" ixy="0" ixz="0" iyy="1e-3" iyz="0" izz="1e-3"/>
     </inertial>
   </link>
@@ -71,7 +59,7 @@
     <parent link="pedestal"/>
     <child link="mid_stomach"/>
-    <origin rpy="0 0 0"  xyz="0 0 0"/>
+    <origin rpy="0 0 0" xyz="0 0 0"/>
   </joint>
-  <xacro:torso side="right" covers="yes" />
+  <xacro:torso side="right" covers="yes"/>
   <joint name="head_tilt" type="revolute">
    <axis xyz="0 1 0"/>
@@ -90,6 +78,6 @@
    <dynamics damping="0.7"/>
   </joint>
-  <xacro:head covers="yes" />
-  <xacro:face covers="yes" />
+  <xacro:head covers="yes"/>
+  <xacro:face covers="yes"/>
   <joint name="face" type="fixed">
     <origin rpy="0 0 0" xyz="0 0.0637 0.079"/>
@@ -97,5 +85,5 @@
     <child link="face"/>
   </joint>
-  <xacro:arm side="right" flip="1" covers="yes" />
+  <xacro:arm side="right" flip="1" covers="yes"/>
   <joint name="right_shoulder_side" type="revolute">
    <axis xyz="0 1 0"/>
@@ -106,5 +94,5 @@
    <dynamics damping="0.7"/>
   </joint>
-  <xacro:rhand side="right" neg="1" covers="yes" />
+  <xacro:rhand side="right" neg="1" covers="yes"/>
   <joint name="right_wrist" type="revolute">
    <axis xyz="0 0 1"/>
@@ -115,5 +103,5 @@
    <dynamics damping="0.7"/>
   </joint>
-  <xacro:arm side="left" flip="-1" covers="yes" />
+  <xacro:arm side="left" flip="-1" covers="yes"/>
   <joint name="left_shoulder_side" type="revolute">
    <axis xyz="0 1 0"/>
@@ -124,5 +112,5 @@
    <dynamics damping="0.7"/>
   </joint>
-  <xacro:lhand side="left" neg="-1" covers="yes" />
+  <xacro:lhand side="left" neg="-1" covers="yes"/>
   <joint name="left_wrist" type="revolute">
    <axis xyz="0 0 1"/>
@@ -133,5 +121,5 @@
    <dynamics damping="0.7"/>
   </joint>
-  <xacro:include filename="$(find inmoov_description)/urdf/sensors.gazebo"/>
+  <xacro:include filename="$(find inmoov_description)/urdf/emr_sensors.gazebo"/>
   <xacro:include filename="$(find inmoov_description)/urdf/servos.urdf.xacro"/>
   <xacro:include filename="$(find inmoov_description)/urdf/materials.gazebo"/>

Commit message: Fixed a few remaining merge conlicts and mistakes.

File: inmoov_description/robots/inmoov.urdf.xacro (robot description, xacro)
@@ -175,10 +175,6 @@
    <child link="left_hand"/>
   </joint>
-<<<<<<< HEAD
-  <xacro:include filename="$(find inmoov_description)/urdf/sensors.gazebo"/>
-=======
   <xacro:include filename="$(find inmoov_description)/urdf/emr_sensors.gazebo"/>
   <xacro:include filename="$(find inmoov_description)/urdf/contact_sensors.gazebo"/>
->>>>>>> 634610668551a6d8b94040087a2017a49e50d6e6
   <xacro:include filename="$(find inmoov_description)/urdf/servos.urdf.xacro"/>
   <xacro:include filename="$(find inmoov_description)/urdf/materials.gazebo"/>

File: inmoov_description/robots/inmoov_no_collision.urdf.xacro (robot description, xacro)
@@ -111,20 +111,4 @@
     </inertial>
   </link>
-  <link name="right_wrist_link">
-    <visual>
-      <geometry>
-        <mesh filename="package://inmoov_meshes/meshes/virtual.stl" scale="0.001 0.001 0.001"/>
-      </geometry>
-      <origin rpy="0 0 0" xyz="0 0 0"/>
-      <material name="cframe">
-        <color rgba="0.25 0.25 0.25 1"/>
-      </material>
-    </visual>
-    <inertial>
-      <origin rpy="0 0 0" xyz="0 0.001 0.001"/>
-      <mass value="5.25e-4"/>
-      <inertia ixx="1e-3"  ixy="0"  ixz="0" iyy="1e-3" iyz="0" izz="1e-3" />
-    </inertial>
-  </link>
   <joint name="right_wrist" type="revolute">
    <axis xyz="0 0 1"/>
@@ -140,9 +124,5 @@
    <child link="right_hand"/>
   </joint>
-<<<<<<< HEAD:inmoov_description/robots/inmoov.xacro
-  <xacro:arm side="left" flip="-1" covers="yes" />
-=======
   <xacro:arm side="left" flip="-1" covers="yes"/>
->>>>>>> 634610668551a6d8b94040087a2017a49e50d6e6:inmoov_description/robots/inmoov_no_collision.urdf.xacro
   <joint name="left_shoulder_side" type="revolute">
    <axis xyz="0 1 0"/>
@@ -170,20 +150,4 @@
     </inertial>
   </link>
-  <link name="left_wrist_link">
-    <visual>
-      <geometry>
-        <mesh filename="package://inmoov_meshes/meshes/virtual.stl" scale="0.001 0.001 0.001"/>
-      </geometry>
-      <origin rpy="0 0 0" xyz="0 0 0"/>
-      <material name="cframe">
-        <color rgba="0.25 0.25 0.25 1"/>
-      </material>
-    </visual>
-    <inertial>
-      <origin rpy="0 0 0" xyz="0 0.001 0.001"/>
-      <mass value="5.25e-4"/>
-      <inertia ixx="1e-3"  ixy="0"  ixz="0" iyy="1e-3" iyz="0" izz="1e-3" />
-    </inertial>
-  </link>
   <joint name="left_wrist" type="revolute">
    <axis xyz="0 0 1"/>
@@ -199,9 +163,5 @@
    <child link="left_hand"/>
   </joint>
-<<<<<<< HEAD:inmoov_description/robots/inmoov.xacro
-  <xacro:include filename="$(find inmoov_description)/urdf/sensors.gazebo"/>
-=======
   <xacro:include filename="$(find inmoov_description)/urdf/emr_sensors.gazebo"/>
->>>>>>> 634610668551a6d8b94040087a2017a49e50d6e6:inmoov_description/robots/inmoov_no_collision.urdf.xacro
   <xacro:include filename="$(find inmoov_description)/urdf/servos.urdf.xacro"/>
   <xacro:include filename="$(find inmoov_description)/urdf/materials.gazebo"/>
